File: lowstepper_hardware/_autosave-lowstepper_hardware.sch (KiCad schematic (older format))
At the start: 41 parts, among them J1 CLOCK_IN, J2 TRIG, J3 RESET, J4 RATE, J5 MORPH, J6 CHUNK, J7 OUT, J8 DONT_FUCK_UP_RED_LINE, Q1 MMBT3904, Q2 MMBT3904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

Commit message: Closer to done hardware, schematics 75% there
Parts:
- C1, C2, C3: footprint (none) -> Capacitor_SMD:C_0805_2012Metric_Pad1.15x1.40mm_HandSolder
- RV1, RV2, RV3: footprint (none) -> Potentiometer_THT:Potentiometer_Alpha_RD901F-40-00D_Single_Vertical
- U2: footprint (none) -> Package_SO:SOIC-14_3.9x8.7mm_P1.27mm
Changed lines of the file:
@@
 F 0 "C2" V 4571 850 50  0000 C CNN
 F 1 "1n" V 4662 850 50  0000 C CNN
-F 2 "" H 4800 850 50  0001 C CNN
+F 2 "Capacitor_SMD:C_0805_2012Metric_Pad1.15x1.40mm_HandSolder" H 4800 850 50  0001 C CNN
 F 3 "~" H 4800 850 50  0001 C CNN
 	1    4800 850
@@
 F 0 "C3" V 4571 2700 50  0000 C CNN
 F 1 "1n" V 4662 2700 50  0000 C CNN
-F 2 "" H 4800 2700 50  0001 C CNN
+F 2 "Capacitor_SMD:C_0805_2012Metric_Pad1.15x1.40mm_HandSolder" H 4800 2700 50  0001 C CNN
 F 3 "~" H 4800 2700 50  0001 C CNN
 	1    4800 2700
@@
 F 0 "C1" V 4521 4450 50  0000 C CNN
 F 1 "1n" V 4612 4450 50  0000 C CNN
-F 2 "" H 4750 4450 50  0001 C CNN
+F 2 "Capacitor_SMD:C_0805_2012Metric_Pad1.15x1.40mm_HandSolder" H 4750 4450 50  0001 C CNN
 F 3 "~" H 4750 4450 50  0001 C CNN
 	1    4750 4450
@@
 F 0 "RV1" V 6853 3150 50  0000 C CNN
 F 1 "10K" V 6944 3150 50  0000 C CNN
-F 2 "" H 7050 3150 50  0001 C CNN
+F 2 "Potentiometer_THT:Potentiometer_Alpha_RD901F-40-00D_Single_Vertical" H 7050 3150 50  0001 C CNN
 F 3 "~" H 7050 3150 50  0001 C CNN
 	1    7050 3150
@@
 F 0 "RV2" V 6853 3800 50  0000 C CNN
 F 1 "10K" V 6944 3800 50  0000 C CNN
-F 2 "" H 7050 3800 50  0001 C CNN
+F 2 "Potentiometer_THT:Potentiometer_Alpha_RD901F-40-00D_Single_Vertical" H 7050 3800 50  0001 C CNN
 F 3 "~" H 7050 3800 50  0001 C CNN
 	1    7050 3800
@@
 F 0 "RV3" V 6853 4450 50  0000 C CNN
 F 1 "10K" V 6944 4450 50  0000 C CNN
-F 2 "" H 7050 4450 50  0001 C CNN
+F 2 "Potentiometer_THT:Potentiometer_Alpha_RD901F-40-00D_Single_Vertical" H 7050 4450 50  0001 C CNN
 F 3 "~" H 7050 4450 50  0001 C CNN
 	1    7050 4450
@@
 F 0 "U2" H 4800 2167 50  0000 C CNN
 F 1 "MCP6004" H 4800 2076 50  0000 C CNN
-F 2 "" H 4750 1900 50  0001 C CNN
+F 2 "Package_SO:SOIC-14_3.9x8.7mm_P1.27mm" H 4750 1900 50  0001 C CNN
 F 3 "http://ww1.microchip.com/downloads/en/DeviceDoc/21733j.pdf" H 4850 2000 50  0001 C CNN
 	1    4800 1800
@@
 F 0 "U2" H 4800 3283 50  0000 C CNN
 F 1 "MCP6004" H 4800 3374 50  0000 C CNN
-F 2 "" H 4750 3750 50  0001 C CNN
+F 2 "Package_SO:SOIC-14_3.9x8.7mm_P1.27mm" H 4750 3750 50  0001 C CNN
 F 3 "http://ww1.microchip.com/downloads/en/DeviceDoc/21733j.pdf" H 4850 3850 50  0001 C CNN
 	2    4800 3650
@@
 F 0 "U2" H 4750 5033 50  0000 C CNN
 F 1 "MCP6004" H 4750 5124 50  0000 C CNN
-F 2 "" H 4700 5500 50  0001 C CNN
+F 2 "Package_SO:SOIC-14_3.9x8.7mm_P1.27mm" H 4700 5500 50  0001 C CNN
 F 3 "http://ww1.microchip.com/downloads/en/DeviceDoc/21733j.pdf" H 4800 5600 50  0001 C CNN
 	3    4750 5400
@@
 F 0 "U2" H 3400 7367 50  0000 C CNN
 F 1 "MCP6004" H 3400 7276 50  0000 C CNN
-F 2 "" H 3350 7100 50  0001 C CNN
+F 2 "Package_SO:SOIC-14_3.9x8.7mm_P1.27mm" H 3350 7100 50  0001 C CNN
 F 3 "http://ww1.microchip.com/downloads/en/DeviceDoc/21733j.pdf" H 3450 7200 50  0001 C CNN
 	4    3400 7000
@@
 F 0 "U2" H 4058 6996 50  0000 L CNN
 F 1 "MCP6004" H 4058 6905 50  0000 L CNN
-F 2 "" H 4050 7050 50  0001 C CNN
+F 2 "Package_SO:SOIC-14_3.9x8.7mm_P1.27mm" H 4050 7050 50  0001 C CNN
 F 3 "http://ww1.microchip.com/downloads/en/DeviceDoc/21733j.pdf" H 4150 7150 50  0001 C CNN
 	5    4100 6950
