File: lowstepper_hardware/_autosave-lowstepper_hardware.sch (KiCad schematic (older format))
At the start: 48 parts, among them J1 CLOCK_IN, J2 TRIG, J3 RESET, J4 RATE, J5 MORPH, J6 CHUNK, J7 OUT, J8 DONT_FUCK_UP_RED_LINE, J9 OUT, Q1 MMBT3904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

Commit message: hardware annotation / PCB placement
Parts:
- removed SW?: SW_Push, symbol Switch:SW_Push
- added SW1: SW_SPST, Button_Switch_SMD:SW_SPST_PTS645, symbol Switch:SW_SPST
Changed lines of the file:
@@
 $EndComp
 $Comp
-L Switch:SW_Push SW?
-U 1 1 60505B87
-P 12300 10150
-F 0 "SW?" H 12300 10435 50  0000 C CNN
-F 1 "SW_Push" H 12300 10344 50  0000 C CNN
-F 2 "" H 12300 10350 50  0001 C CNN
-F 3 "~" H 12300 10350 50  0001 C CNN
-	1    12300 10150
+L Switch:SW_SPST SW1
+U 1 1 6005B351
+P 15700 5250
+F 0 "SW1" H 15700 5485 50  0000 C CNN
+F 1 "SW_SPST" H 15700 5394 50  0000 C CNN
+F 2 "Button_Switch_SMD:SW_SPST_PTS645" H 15700 5250 50  0001 C CNN
+F 3 "~" H 15700 5250 50  0001 C CNN
+	1    15700 5250
 	1    0    0    -1
 $EndComp
