File: daisy_hardware_v1/daisy_hardware_v1.kicad_sch (KiCad schematic)
At the start: 21 parts, among them J1 Conn_02x08_Odd_Even, J2 PJ398SM-12, J3 PJ398SM-12, J4 PJ398SM-12, J5 PJ398SM-12, U1 RAF_DAISY_SEED_V1, U2 TL072, U3 CD4051B, U4 CD4051B, U5 LM4040DBZ-10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

Commit message: first pass of daisy schematic
Parts:
- added RV? (x6): 10k, symbol Device:R_Potentiometer_US
- added SW? (x2): SW_SPST, symbol Switch:SW_SPST
Connections:
- net +3V3: now also RV?.1, RV?.1, RV?.1, RV?.1, RV?.1, RV?.1
- net CV_DIVIDE_A: no longer U7.8
- net CV_DIVIDE_B: now also U7.8
- net CV_MORPH_A: no longer U7.7
- net CV_MORPH_B: now also U7.7
- net CV_RATE_A: no longer U7.1
- net CV_RATE_B: now also U7.1
- net GND: now also RV?.3, RV?.3, RV?.3, RV?.3, RV?.3, RV?.3, SW?.1 (A), SW?.1 (A)
- net POT_DIVIDE_A: now also RV?.2
- net POT_DIVIDE_B: now also RV?.2
- net POT_MORPH_A: now also RV?.2
- net POT_MORPH_B: now also RV?.2
- net POT_RATE_A: now also RV?.2
- net POT_RATE_B: now also RV?.2
- net LOOP_A: now reaches U1.26
- net LOOP_A: now also SW?.2 (B)
- net LOOP_B: now reaches U1.27
- net LOOP_B: now also SW?.2 (B)
- no-connect marks 17 -> 18
Other:
- note added: "CV IN"
- note added: "CV OUT"
- note added: "DAISY"
- note added: "EOC"
- note added: "GATE IN"
- note added: "PERIPHERALS"
- note added: "POTS"
- note added: "POWER"
- note added: "TODO: INLINE LEDS"
- moved on the sheet: C1, C2, C3, C4, J1, J2, J3, J4, J5, R1, R2, R3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
