File: daisy_hardware_v1/daisy_hardware_v1.kicad_sch (KiCad schematic)
At the start: 38 parts, among them J1 Conn_02x08_Odd_Even, J2 PJ398SM-12, J20 Conn_01x18_Female, J21 Conn_01x18_Female, J3 PJ398SM-12, J4 PJ398SM-12, J5 PJ398SM-12, J6 Conn_01x18_Male, J9 Conn_01x18_Male, SW1 SW_SPDT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

Commit message: okay, JLC export time
Parts:
- added C14: 100n, Capacitor_SMD:C_0603_1608Metric, symbol Device:C_Small
- added C15: 10u, Capacitor_SMD:CP_Elec_4x5.3, symbol Device:C_Polarized_Small_US
- added R6: 10k, Resistor_SMD:R_0603_1608Metric, symbol Device:R_Small_US
- added R7: 3.3k, Resistor_SMD:R_0603_1608Metric, symbol Device:R_Small_US
- added U10: LM1117-5.0, Package_TO_SOT_SMD:SOT-223, symbol Regulator_Linear:LM1117-5.0
- C1, C13, C2, C3: footprint Capacitor_SMD:CP_Elec_3x5.3 -> Capacitor_SMD:CP_Elec_4x5.3
Connections:
- net +12V: now also C13.1, U10.3 (VI)
- net +3V3: no longer U3.16 (VCC), U4.16 (VCC)
- net +5V: now also U3.16 (VCC), U4.16 (VCC), C14.1, C15.1, R6.1, U10.2 (VO); no longer C13.1, J1.11 (Pin_11), J1.12 (Pin_12)
- net GND: now also C14.2, C15.2, R7.2, U10.1 (GND)
- net V_bias: now also R6.2, R7.1
- no-connect marks 14 -> 16

Commit message: faceplate and circuit still in same progress, reviewed tho
Parts:
- added D1, D2: LED_Dual_Bidirectional, LED_THT:LED_D5.0mm, symbol Device:LED_Dual_Bidirectional
- added R15, R8: 1k, Resistor_SMD:R_0603_1608Metric, symbol Device:R_Small_US
- added U11: TL072, Package_SO:SOIC-8_3.9x4.9mm_P1.27mm, symbol Amplifier_Operational:TL072
Connections:
- net +12V: now also J20.1 (Pin_1), J6.18 (Pin_18), U11.8 (V+)
- net +3V3: now also U8.8 (V+); no longer U8.4 (V-)
- net -12V: now also J20.18 (Pin_18), J6.1 (Pin_1), U11.4 (V-)
- net DAC1_TOP: now also U11.5 (+)
- net DAC2_TOP: now also U11.3 (+)
- net GND: now also U8.4 (V-), R15.1, R8.1; no longer U8.8 (V+)
- new net: D1.1 (KA), U11.7
- new net: D1.2 (AK), R8.2, U11.6 (-)
- new net: D2.2 (AK), R15.2, U11.2 (-)
- new net: D2.1 (KA), U11.1
Other:
- moved on the sheet: J2, R1, R3, U2B
