File: daisy_hardware_v1/daisy_hardware_v1.kicad_sch (KiCad schematic)
At the start: 48 parts, among them J1 Conn_02x08_Odd_Even, J2 PJ398SM-12, J20 Conn_01x18_Female, J21 Conn_01x18_Female, J3 PJ398SM-12, J4 PJ398SM-12, J5 PJ398SM-12, J6 Conn_01x18_Male, J9 Conn_01x18_Male, SW1 SW_SPDT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

Commit message: another export
Parts:
- removed J1: Conn_02x08_Odd_Even, Connector_PinHeader_2.54mm:PinHeader_2x08_P2.54mm_Vertical, symbol Connector_Generic:Conn_02x08_Odd_Even
- added D3, D4: 1N5819HW, Diode_SMD:D_SOD-123, symbol Device:D_Small_Filled
- added J1: Conn_02x05_Odd_Even, Connector_PinHeader_2.54mm:PinHeader_2x05_P2.54mm_Vertical, symbol Connector_Generic:Conn_02x05_Odd_Even
Connections:
- net +12V: now also D4.1 (K)
- net -12V: now also D3.2 (A)
- net GND: now also J1.3 (Pin_3), J1.4 (Pin_4), J1.5 (Pin_5), J1.6 (Pin_6), J1.7 (Pin_7), J1.8 (Pin_8)
- new net: D3.1 (K), J1.1 (Pin_1), J1.2 (Pin_2)
- new net: D4.2 (A), J1.10 (Pin_10), J1.9 (Pin_9)
- no-connect marks 16 -> 10

Commit message: 3v3a connected
Connections:
- net +3V3: no longer J21.1 (Pin_1), J9.18 (Pin_18), RV1.1, RV2.1, RV3.1, RV4.1, RV5.1, RV6.1, RV7.1, RV8.1
- net 3V3A: now reaches U1.21
- net 3V3A: now also J21.1 (Pin_1), J9.18 (Pin_18), RV1.1, RV2.1, RV3.1, RV4.1, RV5.1, RV6.1, RV7.1, RV8.1
- no-connect marks 10 -> 9
Other:
- note removed: "TODO: INLINE LEDS"
