File: daisy_hardware_v1/_autosave-daisy_hardware_v1.kicad_sch (KiCad schematic)
At the start: 31 parts, among them J1 Conn_02x08_Odd_Even, J2 PJ398SM-12, J3 PJ398SM-12, J4 Connector_Audio:Jack_3.5mm_Qi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, J5 PJ398SM-12, SW1 SW_SPST, SW2 SW_SPST, U1 RAF_DAISY_SEED_V1, U2 TL072, U3 CD4051B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

Commit message: Schematics coming along
Parts:
- gave numbers to parts that had none: 2
Changed lines of the file:
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@@
   (symbol (lib_id "Device:C_Polarized_Small_US") (at 334.01 231.14 0) (unit 1)
     (in_bom yes) (on_board yes) (fields_autoplaced)
-    (property "Reference" "C?" (id 0) (at 336.3214 229.7997 0)
+    (property "Reference" "C2" (id 0) (at 336.3214 229.7997 0)
       (effects (font (size 1.27 1.27)) (justify left))
     )
@@
   (symbol (lib_id "Device:C_Polarized_Small_US") (at 321.31 231.14 0) (unit 1)
     (in_bom yes) (on_board yes) (fields_autoplaced)
-    (property "Reference" "C?" (id 0) (at 323.6214 229.7997 0)
+    (property "Reference" "C1" (id 0) (at 323.6214 229.7997 0)
       (effects (font (size 1.27 1.27)) (justify left))
     )
@@
       (reference "#PWR0189") (unit 1) (value "GND") (footprint "")
     )
+    (path "/ee028d49-2036-48df-8a86-63c94a641d39"
+      (reference "C1") (unit 1) (value "47u") (footprint "Capacitor_SMD:CP_Elec_3x5.3")
+    )
+    (path "/7c3685ea-5658-43d0-9983-d9fb19ca9a38"
+      (reference "C2") (unit 1) (value "47u") (footprint "Capacitor_SMD:CP_Elec_3x5.3")
+    )
     (path "/5cc6cebf-9c38-45c9-91f0-1d41cb67a9b3"
       (reference "C4") (unit 1) (value "10u") (footprint "")
@@
       (reference "C12") (unit 1) (value "1n") (footprint "")
     )
-    (path "/7c3685ea-5658-43d0-9983-d9fb19ca9a38"
-      (reference "C?") (unit 1) (value "47u") (footprint "Capacitor_SMD:CP_Elec_3x5.3")
-    )
-    (path "/ee028d49-2036-48df-8a86-63c94a641d39"
-      (reference "C?") (unit 1) (value "47u") (footprint "Capacitor_SMD:CP_Elec_3x5.3")
-    )
     (path "/e8365b2a-3ef6-404e-a2ae-9e53aa232c16"
